Commit message: physical move update

File: code-v2/nesyrl/nesyrl/envs/physical/models/objects/goal_area.urdf (robot description, URDF)
Before this commit: robot cube, 1 links, 0 joints
Links:
- link base_link: geometry visual box size=.05 .05 .05

File: code-v2/nesyrl/nesyrl/envs/physical/models/robots/nico/nico_upper_rh6d.urdf (robot description, URDF)
Before this commit: robot nico_upper_rh6d, 12 links, 11 joints
Joints:
- joint r_shoulder_z_rjoint: limit lower=-0.3490 upper=1.3963 effort=30 velocity=1 -> lower=-0.2200 upper=1.3220 effort=30 velocity=1
- joint r_wrist_x_rjoint: type revolute -> fixed
- joint r_wrist_z_rjoint: limit lower=-1.571 upper=1.571 effort=30 velocity=1 -> lower=-3.142 upper=0 effort=30 velocity=1; origin xyz=0 0 -0.105 rpy=0 0 1.57 -> xyz=0 0 -0.105 rpy=0 0 3.142; type revolute -> fixed
